Commit message: 25/09/24

File: src/franka_ros/franka_description/robots/panda_arm.urdf.xacro (robot description, xacro)
@@ -3,5 +3,5 @@
   <xacro:arg name="arm_id" default="panda" /> <!-- Name of this panda -->
   <xacro:arg name="hand"   default="false" /> <!-- Should a franka_gripper be mounted at the flange?" -->
-  <xacro:arg name="gazebo" default="false" /> <!-- Is the robot being simulated in gazebo?" -->
+  <xacro:arg name="gazebo" default="true" /> <!-- Is the robot being simulated in gazebo?" -->
   <xacro:property name="arm_id" value="$(arg arm_id)" />
   <xacro:unless value="$(arg gazebo)">

File: src/realsense-ros/realsense2_description/urdf/test_d435_camera.urdf.xacro (robot description, xacro)
@@ -5,7 +5,9 @@
   <xacro:arg name="use_mesh" default="true" />
   <xacro:include filename="$(find realsense2_description)/urdf/_d435.urdf.xacro" />
+  <xacro:arg name="xyz" default="0 0 0" />
+  <xacro:arg name="rpy" default="0 0 0" />
   <link name="base_link" />
   <xacro:sensor_d435 parent="base_link" use_nominal_extrinsics="$(arg use_nominal_extrinsics)" add_plug="$(arg add_plug)" use_mesh="$(arg use_mesh)">
-    <origin xyz="0 0 0" rpy="0 0 0"/>
+    <origin xyz="$(arg xyz)" rpy="$(arg rpy)"/>
   </xacro:sensor_d435>
 </robot>
